File: esc.brd (EAGLE design)
At the start: 98.7 x 39.3 mm, 61 parts, among them IC1 78L05F, Q1 16 MHz, T1 IRFR1205, T2 IRFR1205, T3 IRFR1205, T4 IRFR1205, T5 IRFR1205, T6 IRFR1205, U1 ATMEGA48-20AU

Commit message: Added value to r1 and tRestrict under Quarz
Parts:
- R1: value 10 -> 10k
Changed lines of the file:
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@@
 <layer number="19" name="Unrouted" color="6" fill="1" visible="yes" active="yes"/>
 <layer number="20" name="Dimension" color="15" fill="1" visible="yes" active="yes"/>
-<layer number="21" name="tPlace" color="7" fill="1" visible="no" active="yes"/>
+<layer number="21" name="tPlace" color="7" fill="1" visible="yes" active="yes"/>
 <layer number="22" name="bPlace" color="7" fill="1" visible="no" active="yes"/>
-<layer number="23" name="tOrigins" color="15" fill="1" visible="no" active="yes"/>
+<layer number="23" name="tOrigins" color="15" fill="1" visible="yes" active="yes"/>
 <layer number="24" name="bOrigins" color="15" fill="1" visible="no" active="yes"/>
 <layer number="25" name="tNames" color="7" fill="1" visible="no" active="yes"/>
@@
 <layer number="39" name="tKeepout" color="4" fill="11" visible="no" active="yes"/>
 <layer number="40" name="bKeepout" color="1" fill="11" visible="no" active="yes"/>
-<layer number="41" name="tRestrict" color="4" fill="10" visible="no" active="yes"/>
+<layer number="41" name="tRestrict" color="4" fill="10" visible="yes" active="yes"/>
 <layer number="42" name="bRestrict" color="1" fill="10" visible="no" active="yes"/>
 <layer number="43" name="vRestrict" color="2" fill="10" visible="no" active="yes"/>
@@
 <layer number="49" name="Reference" color="7" fill="1" visible="no" active="yes"/>
 <layer number="50" name="dxf" color="7" fill="1" visible="no" active="yes"/>
-<layer number="51" name="tDocu" color="7" fill="1" visible="no" active="yes"/>
+<layer number="51" name="tDocu" color="7" fill="1" visible="yes" active="yes"/>
 <layer number="52" name="bDocu" color="7" fill="1" visible="no" active="yes"/>
 <layer number="91" name="Nets" color="2" fill="1" visible="no" active="no"/>
@@
 <rectangle x1="69.85" y1="31.75" x2="74.93" y2="36.83" layer="41"/>
 <rectangle x1="74.93" y1="31.75" x2="77.47" y2="33.9725" layer="41"/>
+<rectangle x1="46.99" y1="31.75" x2="54.61" y2="34.29" layer="41"/>
 </plain>
 <attributes>
@@
 <element name="C4" library="rcl" package="C1206" value="100nF" x="42.545" y="7.62" rot="R270"/>
 <element name="C5" library="rcl" package="C1206" value="100nF" x="40.005" y="7.62" rot="R270"/>
-<element name="R1" library="rcl" package="R1206" value="10" x="37.465" y="7.62" rot="R90"/>
+<element name="R1" library="rcl" package="R1206" value="10k" x="37.465" y="7.62" rot="R90"/>
 <element name="R2" library="rcl" package="R1206" value="10k" x="71.12" y="20.32" rot="R180"/>
 <element name="X1" library="con-wago-500" package="W237-102" value="" x="92.71" y="19.05" rot="R90">

Commit message: ISP mirror
Parts:
- flipped SV1 to the bottom
Routing:
- net SCK: track 37.4 -> 47.7 mm
- net MISO: track 36.9 -> 42.7 mm
- net VCC: track 126.8 -> 127.7 mm, vias 4 -> 6
- net MOSI: track 37.9 -> 38.4 mm
Changed lines of the file:
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@@
 <layer number="14" name="Route14" color="1" fill="6" visible="no" active="no"/>
 <layer number="15" name="Route15" color="4" fill="6" visible="no" active="no"/>
-<layer number="16" name="Bottom" color="1" fill="1" visible="no" active="yes"/>
+<layer number="16" name="Bottom" color="1" fill="1" visible="yes" active="yes"/>
 <layer number="17" name="Pads" color="2" fill="1" visible="yes" active="yes"/>
 <layer number="18" name="Vias" color="2" fill="1" visible="yes" active="yes"/>
@@
 <rectangle x1="91.44" y1="30.7975" x2="96.52" y2="34.29" layer="41"/>
 <rectangle x1="95.25" y1="34.29" x2="96.52" y2="35.56" layer="41"/>
-<rectangle x1="69.85" y1="31.75" x2="74.93" y2="36.83" layer="41"/>
-<rectangle x1="74.93" y1="31.75" x2="77.47" y2="33.9725" layer="41"/>
 <rectangle x1="46.99" y1="31.75" x2="54.61" y2="34.29" layer="41"/>
 </plain>
@@
 </class>
 </classes>
-<designrules name="designRules-2015-03 *">
+<designrules name="designRules-2015-03">
 <description language="de">&lt;b&gt;EAGLE Design Rules&lt;/b&gt;
 &lt;p&gt;
@@
 <element name="R20" library="rcl" package="R1206" value="180" x="62.23" y="24.765"/>
 <element name="LED1" library="led" package="CHIPLED_1206" value="" x="67.945" y="26.9875" rot="R270"/>
-<element name="SV1" library="con-ml" package="ML6" value="" x="73.66" y="34.29">
-<attribute name="OC_NEWARK" value="unknown" x="73.66" y="34.29" size="1.778" layer="27" display="off"/>
-<attribute name="MPN" value="" x="73.66" y="34.29" size="1.778" layer="27" display="off"/>
-<attribute name="MF" value="" x="73.66" y="34.29" size="1.778" layer="27" display="off"/>
-<attribute name="OC_FARNELL" value="unknown" x="73.66" y="34.29" size="1.778" layer="27" display="off"/>
+<element name="SV1" library="con-ml" package="ML6" value="" x="73.66" y="34.29" rot="MR0">
+<attribute name="OC_NEWARK" value="unknown" x="73.66" y="34.29" size="1.778" layer="28" rot="MR0" display="off"/>
+<attribute name="MPN" value="" x="73.66" y="34.29" size="1.778" layer="28" rot="MR0" display="off"/>
+<attribute name="MF" value="" x="73.66" y="34.29" size="1.778" layer="28" rot="MR0" display="off"/>
+<attribute name="OC_FARNELL" value="unknown" x="73.66" y="34.29" size="1.778" layer="28" rot="MR0" display="off"/>
 </element>
 <element name="SV2" library="con-ml" package="ML6" value="" x="93.98" y="31.75" rot="R90">
@@
 <wire x1="83.109" y1="21.184" x2="83.109" y2="24.819" width="0.4064" layer="1"/>
 <wire x1="83.109" y1="24.819" x2="83.69" y2="24.13" width="0.4064" layer="1"/>
-<wire x1="71.12" y1="35.56" x2="64.64" y2="35.56" width="0.4064" layer="1"/>
-<wire x1="64.64" y1="35.56" x2="63.59375" y2="34.51375" width="0.4064" layer="1"/>
-<wire x1="63.59375" y1="34.51375" x2="57.02" y2="27.94" width="0.4064" layer="1"/>
-<wire x1="72.542" y1="20.32" x2="72.542" y2="21.4245" width="0.4064" layer="1"/>
-<wire x1="72.542" y1="21.4245" x2="73.66" y2="22.5425" width="0.4064" layer="1"/>
-<via x="73.66" y="22.5425" extent="1-16" drill="0.8"/>
-<wire x1="73.66" y1="22.5425" x2="73.66" y2="22.86" width="0.4064" layer="16"/>
-<wire x1="78.105" y1="27.305" x2="78.105" y2="28.2575" width="0.4064" layer="16"/>
-<wire x1="78.105" y1="28.2575" x2="77.1525" y2="29.21" width="0.4064" layer="16"/>
-<wire x1="77.1525" y1="29.21" x2="68.8975" y2="29.21" width="0.4064" layer="16"/>
-<wire x1="68.8975" y1="29.21" x2="65.0875" y2="33.02" width="0.4064" layer="16"/>
-<via x="65.0875" y="33.02" extent="1-16" drill="0.8"/>
-<wire x1="65.0875" y1="33.02" x2="63.59375" y2="34.51375" width="0.4064" layer="1"/>
-<wire x1="73.66" y1="22.86" x2="78.105" y2="27.305" width="0.4064" layer="16"/>
 <wire x1="75.565" y1="19.05" x2="74.3835" y2="20.2315" width="0.4064" layer="1"/>
 <wire x1="74.3835" y1="20.2315" x2="74.6125" y2="20.2315" width="0.4064" layer="1"/>
@@
 <wire x1="35.2425" y1="9.525" x2="35.2425" y2="9.2075" width="0.4064" layer="16"/>
 <wire x1="35.2425" y1="9.2075" x2="39.0525" y2="5.3975" width="0.4064" layer="16"/>
+<wire x1="83.109" y1="24.819" x2="83.239" y2="24.819" width="0.4064" layer="1"/>
+<wire x1="83.239" y1="24.819" x2="85.09" y2="26.67" width="0.4064" layer="1"/>
+<via x="85.09" y="26.67" extent="1-16" drill="0.8"/>
+<wire x1="85.09" y1="26.67" x2="85.09" y2="30.48" width="0.4064" layer="16"/>
+<wire x1="85.09" y1="30.48" x2="80.01" y2="35.56" width="0.4064" layer="16"/>
+<via x="80.01" y="35.56" extent="1-16" drill="0.8"/>
+<wire x1="80.01" y1="35.56" x2="76.2" y2="35.56" width="0.4064" layer="1"/>
+<wire x1="56.8325" y1="27.7525" x2="56.8325" y2="28.8925" width="0.4064" layer="1"/>
+<wire x1="56.8325" y1="28.8925" x2="59.69" y2="31.75" width="0.4064" layer="1"/>
+<via x="59.69" y="31.75" extent="1-16" drill="0.8"/>
+<wire x1="59.69" y1="31.75" x2="59.69" y2="30.48" width="0.4064" layer="16"/>
+<wire x1="59.69" y1="30.48" x2="69.85" y2="20.32" width="0.4064" layer="16"/>
+<wire x1="69.85" y1="20.32" x2="71.755" y2="20.32" width="0.4064" layer="16"/>
+<wire x1="71.755" y1="20.32" x2="73.66" y2="22.225" width="0.4064" layer="16"/>
+<via x="73.66" y="22.225" extent="1-16" drill="0.8"/>
+<wire x1="73.66" y1="22.225" x2="72.39" y2="20.955" width="0.4064" layer="1"/>
+<wire x1="72.39" y1="20.955" x2="72.39" y2="20.472" width="0.4064" layer="1"/>
+<wire x1="72.39" y1="20.472" x2="72.542" y2="20.32" width="0.4064" layer="1"/>
 </signal>
 <signal name="N$1">
@@
 <wire x1="22.5425" y1="11.1125" x2="22.5425" y2="12.065" width="0.4064" layer="1"/>
 <wire x1="22.5425" y1="12.065" x2="21.9075" y2="12.7" width="0.4064" layer="1"/>
+<wire x1="54.74" y1="27.94" x2="59.82" y2="27.94" width="0" layer="19" extent="1-1"/>
 </signal>
 <signal name="N$2">
@@
 <wire x1="50.165" y1="16.1925" x2="57.15" y2="23.1775" width="0.4064" layer="16"/>
 <via x="57.15" y="23.1775" extent="1-16" drill="0.8"/>
-<wire x1="69.215" y1="34.29" x2="61.2775" y2="26.3525" width="0.4064" layer="1"/>
 <wire x1="61.2775" y1="26.3525" x2="59.69" y2="26.3525" width="0.4064" layer="1"/>
 <wire x1="59.69" y1="26.3525" x2="59.055" y2="25.7175" width="0.4064" layer="1"/>
 <wire x1="59.055" y1="25.7175" x2="59.055" y2="25.0825" width="0.4064" layer="1"/>
 <wire x1="59.055" y1="25.0825" x2="57.15" y2="23.1775" width="0.4064" layer="1"/>
-<wire x1="69.215" y1="34.29" x2="72.39" y2="34.29" width="0.4064" layer="1"/>
-<wire x1="72.39" y1="34.29" x2="73.66" y2="35.56" width="0.4064" layer="1"/>
+<wire x1="61.2775" y1="26.3525" x2="69.215" y2="34.29" width="0.4064" layer="1"/>
+<wire x1="69.215" y1="34.29" x2="73.3425" y2="34.29" width="0.4064" layer="1"/>
+<wire x1="73.3425" y1="34.29" x2="73.66" y2="34.6075" width="0.4064" layer="1"/>
+<wire x1="73.66" y1="34.6075" x2="73.66" y2="35.56" width="0.4064" layer="1"/>
 </signal>
 <signal name="MISO">
@@
 <wire x1="60.96" y1="22.225" x2="62.23" y2="23.495" width="0.4064" layer="1"/>
 <wire x1="62.23" y1="23.495" x2="62.23" y2="26.035" width="0.4064" layer="1"/>
-<wire x1="62.23" y1="26.035" x2="69.215" y2="33.02" width="0.4064" layer="1"/>
-<wire x1="69.215" y1="33.02" x2="71.12" y2="33.02" width="0.4064" layer="1"/>
+<wire x1="62.23" y1="26.035" x2="66.675" y2="30.48" width="0.4064" layer="1"/>
+<wire x1="76.2" y1="33.02" x2="76.2" y2="31.75" width="0.4064" layer="1"/>
+<wire x1="76.2" y1="31.75" x2="74.93" y2="30.48" width="0.4064" layer="1"/>
+<wire x1="74.93" y1="30.48" x2="66.675" y2="30.48" width="0.4064" layer="1"/>
 </signal>
 <signal name="SCK">
@@
 <wire x1="62.5475" y1="21.9075" x2="63.8175" y2="21.9075" width="0.4064" layer="1"/>
 <wire x1="63.8175" y1="21.9075" x2="67.945" y2="26.035" width="0.4064" layer="1"/>
-<wire x1="67.945" y1="26.035" x2="67.945" y2="28.2575" width="0.4064" layer="1"/>
-<wire x1="73.66" y1="33.3375" x2="73.66" y2="33.02" width="0.4064" layer="16"/>
-<wire x1="67.945" y1="28.2575" x2="68.58" y2="28.8925" width="0.4064" layer="1"/>
-<wire x1="68.58" y1="28.8925" x2="69.5325" y2="28.8925" width="0.4064" layer="1"/>
-<wire x1="69.5325" y1="28.8925" x2="73.66" y2="33.02" width="0.4064" layer="1"/>
+<wire x1="67.945" y1="26.035" x2="67.945" y2="27.94" width="0.4064" layer="1"/>
+<wire x1="67.945" y1="27.94" x2="68.58" y2="28.575" width="0.4064" layer="1"/>
+<wire x1="68.58" y1="28.575" x2="74.295" y2="28.575" width="0.4064" layer="1"/>
+<wire x1="74.295" y1="28.575" x2="78.105" y2="32.385" width="0.4064" layer="1"/>
+<wire x1="78.105" y1="32.385" x2="78.105" y2="33.9725" width="0.4064" layer="1"/>
+<wire x1="78.105" y1="33.9725" x2="77.7875" y2="34.29" width="0.4064" layer="1"/>
+<wire x1="77.7875" y1="34.29" x2="74.93" y2="34.29" width="0.4064" layer="1"/>
+<wire x1="74.93" y1="34.29" x2="73.66" y2="33.02" width="0.4064" layer="1"/>
 </signal>
 <signal name="RESET">
@@
 <wire x1="56.556771875" y1="19.084428125" x2="68.393571875" y2="19.084428125" width="0.4064" layer="1"/>
 <wire x1="68.393571875" y1="19.084428125" x2="69.698" y2="20.32" width="0.4064" layer="1"/>
-<wire x1="69.698" y1="20.32" x2="69.698" y2="21.1205" width="0.4064" layer="1"/>
-<wire x1="69.698" y1="21.1205" x2="71.12" y2="22.5425" width="0.4064" layer="1"/>
-<via x="71.12" y="22.5425" extent="1-16" drill="0.8"/>
-<via x="76.2" y="27.6225" extent="1-16" drill="0.8"/>
-<wire x1="76.2" y1="27.6225" x2="76.2" y2="33.02" width="0.4064" layer="1"/>
-<wire x1="76.2" y1="27.6225" x2="71.12" y2="22.5425" width="0.4064" layer="16"/>
+<wire x1="71.12" y1="33.02" x2="69.85" y2="33.02" width="0.4064" layer="1"/>
+<wire x1="69.85" y1="33.02" x2="68.58" y2="31.75" width="0.4064" layer="1"/>
+<via x="68.58" y="31.75" extent="1-16" drill="0.8"/>
+<wire x1="68.58" y1="31.75" x2="68.58" y2="24.13" width="0.4064" layer="16"/>
+<wire x1="68.58" y1="24.13" x2="70.485" y2="22.225" width="0.4064" layer="16"/>
+<via x="70.485" y="22.225" extent="1-16" drill="0.8"/>
+<wire x1="70.485" y1="22.225" x2="69.85" y2="21.59" width="0.4064" layer="1"/>
+<wire x1="69.85" y1="21.59" x2="69.698" y2="20.32" width="0.4064" layer="1"/>
 </signal>
 <signal name="N$7">
