File: esc.sch (EAGLE design)
At the start: 61 parts, among them IC1 78L05F, Q1 16 MHz, T1 IRFR1205, T2 IRFR1205, T3 IRFR1205, T4 IRFR1205, T5 IRFR1205, T6 IRFR1205, U1 ATMEGA48-20AU

Commit message: esc3 initial commit
Parts:
- removed SV2: (no value), con-ml:ML6
- removed X1: (no value), con-wago-500:W237-102
- removed X2: (no value), con-wago-500:W237-103
- added PAD1, PAD2, PAD4, PAD5, PAD6: WIREPADSMD5-2,5, wirepad:WIREPADSMD5-2,5
- added SV3, SV4: (no value), con-lstb:MA03-1
Connections:
- net GND: now also PAD2.P, SV3.1; no longer SV2.1, SV2.2, X1-2.KL
- net PHASE_A: now also PAD6.P; no longer X2-3.KL
- net PHASE_B: now also PAD4.P; no longer X2-2.KL
- net PHASE_C: now also PAD5.P; no longer X2-1.KL
- net PPM: now also SV4.3
- net RXD: now also SV3.2; no longer SV2.3
- net SCL: now also SV4.1; no longer SV2.6
- net SDA: now also SV4.2; no longer SV2.4
- net TXD: now also SV3.3; no longer SV2.5
- net VSS: now also PAD1.P; no longer X1-1.KL
Changed lines of the file:
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@@
 <part name="R2" library="rcl" deviceset="R-EU_" device="R1206" value="10k"/>
 <part name="P+2" library="supply1" deviceset="VCC" device=""/>
-<part name="X1" library="con-wago-500" deviceset="W237-102" device=""/>
 <part name="C6" library="rcl" deviceset="CPOL-EU" device="E5-10.5" value="470µF"/>
 <part name="C7" library="rcl" deviceset="C-EU" device="C1206" value="100nF"/>
@@
 <part name="GND16" library="supply1" deviceset="GND" device=""/>
 <part name="P+4" library="supply1" deviceset="VCC" device=""/>
-<part name="SV2" library="con-ml" deviceset="ML6" device="">
-<attribute name="MF" value=""/>
-<attribute name="MPN" value=""/>
-<attribute name="OC_FARNELL" value="unknown"/>
-<attribute name="OC_NEWARK" value="unknown"/>
-</part>
-<part name="GND17" library="supply1" deviceset="GND" device=""/>
 <part name="GND18" library="supply1" deviceset="GND" device=""/>
-<part name="X2" library="con-wago-500" deviceset="W237-103" device=""/>
 <part name="C19" library="rcl" deviceset="C-EU" device="C1206" value="1µF"/>
 <part name="C20" library="rcl" deviceset="C-EU" device="C1206" value="1µF"/>
@@
 <part name="R22" library="rcl" deviceset="R-EU_" device="R1206" value="1k"/>
 <part name="R23" library="rcl" deviceset="R-EU_" device="R1206" value="1k"/>
+<part name="PAD1" library="wirepad" deviceset="WIREPAD" device="SMD5-2,5"/>
+<part name="PAD2" library="wirepad" deviceset="WIREPAD" device="SMD5-2,5"/>
+<part name="PAD4" library="wirepad" deviceset="WIREPAD" device="SMD5-2,5"/>
+<part name="PAD5" library="wirepad" deviceset="WIREPAD" device="SMD5-2,5"/>
+<part name="PAD6" library="wirepad" deviceset="WIREPAD" device="SMD5-2,5"/>
+<part name="SV3" library="con-lstb" deviceset="MA03-1" device=""/>
+<part name="SV4" library="con-lstb" deviceset="MA03-1" device=""/>
 </parts>
 <sheets>
@@
 <instance part="R2" gate="G$1" x="76.2" y="73.66" rot="R180"/>
 <instance part="P+2" gate="VCC" x="88.9" y="73.66" rot="R270"/>
-<instance part="X1" gate="-1" x="-22.86" y="124.46"/>
-<instance part="X1" gate="-2" x="-22.86" y="116.84"/>
 <instance part="C6" gate="G$1" x="-7.62" y="121.92"/>
 <instance part="C7" gate="G$1" x="7.62" y="119.38" rot="R180"/>
@@
 <instance part="GND16" gate="1" x="137.16" y="-40.64" rot="R270"/>
 <instance part="P+4" gate="VCC" x="134.62" y="-45.72" rot="R90"/>
-<instance part="SV2" gate="1" x="154.94" y="-60.96"/>
-<instance part="GND17" gate="1" x="127" y="-63.5" rot="R270"/>
-<instance part="GND18" gate="1" x="182.88" y="-63.5" rot="R90"/>
-<instance part="X2" gate="-1" x="287.02" y="45.72" rot="R180"/>
-<instance part="X2" gate="-2" x="287.02" y="50.8" rot="R180"/>
-<instance part="X2" gate="-3" x="287.02" y="55.88" rot="R180"/>
+<instance part="GND18" gate="1" x="190.5" y="-27.94" rot="R90"/>
 <instance part="C19" gate="G$1" x="182.88" y="114.3"/>
 <instance part="C20" gate="G$1" x="182.88" y="58.42"/>
@@
 <instance part="R22" gate="G$1" x="-10.16" y="60.96" rot="R180"/>
 <instance part="R23" gate="G$1" x="-15.24" y="27.94" rot="R180"/>
+<instance part="PAD1" gate="G$1" x="-20.32" y="124.46"/>
+<instance part="PAD2" gate="G$1" x="-20.32" y="116.84"/>
+<instance part="PAD4" gate="G$1" x="284.48" y="50.8" rot="R180"/>
+<instance part="PAD5" gate="G$1" x="284.48" y="45.72" rot="R180"/>
+<instance part="PAD6" gate="G$1" x="284.48" y="55.88" rot="R180"/>
+<instance part="SV3" gate="G$1" x="162.56" y="-25.4"/>
+<instance part="SV4" gate="G$1" x="119.38" y="-25.4"/>
 </instances>
 <busses>
@@
 </segment>
 <segment>
-<pinref part="X1" gate="-2" pin="KL"/>
 <pinref part="C6" gate="G$1" pin="-"/>
 <wire x1="-17.78" y1="116.84" x2="-7.62" y2="116.84" width="0.1524" layer="91"/>
@@
 <pinref part="C10" gate="G$1" pin="2"/>
 <junction x="50.8" y="116.84"/>
+<pinref part="PAD2" gate="G$1" pin="P"/>
 </segment>
 <segment>
@@
 </segment>
 <segment>
-<pinref part="SV2" gate="1" pin="2"/>
-<wire x1="129.54" y1="-63.5" x2="147.32" y2="-63.5" width="0.1524" layer="91"/>
-<pinref part="GND17" gate="1" pin="GND"/>
-</segment>
-<segment>
-<pinref part="SV2" gate="1" pin="1"/>
-<wire x1="162.56" y1="-63.5" x2="180.34" y2="-63.5" width="0.1524" layer="91"/>
+<wire x1="170.18" y1="-27.94" x2="187.96" y2="-27.94" width="0.1524" layer="91"/>
 <pinref part="GND18" gate="1" pin="GND"/>
+<pinref part="SV3" gate="G$1" pin="1"/>
 </segment>
 </net>
@@
 <net name="VSS" class="0">
 <segment>
-<pinref part="X1" gate="-1" pin="KL"/>
 <pinref part="C6" gate="G$1" pin="+"/>
 <wire x1="-17.78" y1="124.46" x2="-7.62" y2="124.46" width="0.1524" layer="91"/>
@@
 <pinref part="VSS1" gate="G$1" pin="VSS"/>
 <wire x1="7.62" y1="124.46" x2="7.62" y2="129.54" width="0.1524" layer="91"/>
+<pinref part="PAD1" gate="G$1" pin="P"/>
 </segment>
 <segment>
@@
 <wire x1="213.36" y1="109.22" x2="276.86" y2="109.22" width="0.1524" layer="91"/>
 <wire x1="276.86" y1="109.22" x2="276.86" y2="55.88" width="0.1524" layer="91"/>
-<pinref part="X2" gate="-3" pin="KL"/>
 <wire x1="276.86" y1="55.88" x2="281.94" y2="55.88" width="0.1524" layer="91"/>
 <pinref part="C19" gate="G$1" pin="2"/>
 <junction x="182.88" y="109.22"/>
+<pinref part="PAD6" gate="G$1" pin="P"/>
 </segment>
 <segment>
@@
 <label x="248.92" y="53.34" size="1.778" layer="95" rot="R180"/>
 <wire x1="259.08" y1="53.34" x2="259.08" y2="50.8" width="0.1524" layer="91"/>
-<pinref part="X2" gate="-2" pin="KL"/>
 <wire x1="259.08" y1="50.8" x2="281.94" y2="50.8" width="0.1524" layer="91"/>
 <pinref part="C20" gate="G$1" pin="2"/>
 <junction x="182.88" y="53.34"/>
+<pinref part="PAD4" gate="G$1" pin="P"/>
 </segment>
 <segment>
@@
 <junction x="213.36" y="-2.54"/>
 <label x="248.92" y="-2.54" size="1.778" layer="95" rot="R180"/>
-<pinref part="X2" gate="-1" pin="KL"/>
 <wire x1="281.94" y1="45.72" x2="269.24" y2="45.72" width="0.1524" layer="91"/>
 <wire x1="269.24" y1="45.72" x2="269.24" y2="-2.54" width="0.1524" layer="91"/>
@@
 <pinref part="C21" gate="G$1" pin="2"/>
 <junction x="182.88" y="-2.54"/>
+<pinref part="PAD5" gate="G$1" pin="P"/>
 </segment>
 <segment>
@@
 <label x="68.58" y="81.28" size="1.778" layer="95"/>
 </segment>
+<segment>
+<wire x1="132.08" y1="-22.86" x2="127" y2="-22.86" width="0.1524" layer="91"/>
+<pinref part="SV4" gate="G$1" pin="3"/>
+<label x="134.62" y="-22.86" size="1.778" layer="95"/>
+</segment>
 </net>
 <net name="SDA" class="0">
@@
 </segment>
 <segment>
-<pinref part="SV2" gate="1" pin="4"/>
-<wire x1="142.24" y1="-60.96" x2="147.32" y2="-60.96" width="0.1524" layer="91"/>
-<label x="139.7" y="-60.96" size="1.778" layer="95" rot="R180"/>
+<wire x1="132.08" y1="-25.4" x2="127" y2="-25.4" width="0.1524" layer="91"/>
+<label x="134.62" y="-25.4" size="1.778" layer="95"/>
+<pinref part="SV4" gate="G$1" pin="2"/>
 </segment>
 </net>
@@
 </segment>
 <segment>
-<pinref part="SV2" gate="1" pin="6"/>
-<wire x1="142.24" y1="-58.42" x2="147.32" y2="-58.42" width="0.1524" layer="91"/>
-<label x="139.7" y="-58.42" size="1.778" layer="95" rot="R180"/>
+<wire x1="132.08" y1="-27.94" x2="127" y2="-27.94" width="0.1524" layer="91"/>
+<label x="134.62" y="-27.94" size="1.778" layer="95"/>
+<pinref part="SV4" gate="G$1" pin="1"/>
 </segment>
 </net>
@@
 </segment>
 <segment>
-<pinref part="SV2" gate="1" pin="3"/>
-<wire x1="162.56" y1="-60.96" x2="167.64" y2="-60.96" width="0.1524" layer="91"/>
-<label x="170.18" y="-60.96" size="1.778" layer="95"/>
+<wire x1="170.18" y1="-25.4" x2="175.26" y2="-25.4" width="0.1524" layer="91"/>
+<label x="177.8" y="-25.4" size="1.778" layer="95"/>
+<pinref part="SV3" gate="G$1" pin="2"/>
 </segment>
 </net>
@@
 </segment>
 <segment>
-<pinref part="SV2" gate="1" pin="5"/>
-<wire x1="167.64" y1="-58.42" x2="162.56" y2="-58.42" width="0.1524" layer="91"/>
-<label x="170.18" y="-58.42" size="1.778" layer="95"/>
-</segment>
-</net>
+<wire x1="175.26" y1="-22.86" x2="170.18" y2="-22.86" width="0.1524" layer="91"/>
+<label x="177.8" y="-22.86" size="1.778" layer="95"/>
+<pinref part="SV3" gate="G$1" pin="3"/>
+</segment>
+</net>
